Commit message: added ixtion to torso

File: rb1_torso_description/robots/rb1_torso.urdf.xacro (robot description, xacro)
@@ -8,5 +8,5 @@
 	<xacro:include filename="$(find rb1_torso_description)/urdf/rb1_torso_3dof.urdf.xacro" />
 	<!-- Import all available sensors -->
-	<!-- xacro:include filename="$(find rb1_torso_description)/urdf/sensors/all_sensors.urdf.xacro" / -->
+	<xacro:include filename="$(find rb1_torso_description)/urdf/sensors/all_sensors.urdf.xacro" />
 	<!-- ***************** -->
 	<!-- Global parameters -->
@@ -15,6 +15,10 @@
 	<!-- Flag to select the high or low quality model -->
 	<xacro:property name="hq" value="true" />
-	<!-- RB-1 arm -->
+	<!-- RB-1 torso -->
 	<xacro:rb1_torso_3dof name="rb1_torso_3dof" hq="${hq}" />
+	<!-- Ixtion sensor in head -->
+	<xacro:sensor_asus_xtion_pro name="xtion_head" parent="link2_head_rb1_torso">
+        <origin xyz="0.055 0.000 0.028" rpy="0 0 0"/>
+   </xacro:sensor_asus_xtion_pro>
 	<!-- Gazebo ros control plugins -->
 	<xacro:ros_control/>

Commit message: changed joint and link names, added transmission

File: rb1_torso_description/robots/rb1_torso.urdf.xacro (robot description, xacro)
@@ -18,5 +18,5 @@
 	<xacro:rb1_torso_3dof name="rb1_torso_3dof" hq="${hq}" />
 	<!-- Ixtion sensor in head -->
-	<xacro:sensor_asus_xtion_pro name="xtion_head" parent="link2_head_rb1_torso">
+	<xacro:sensor_asus_xtion_pro name="xtion_head" parent="link2_head">
         <origin xyz="0.055 0.000 0.028" rpy="0 0 0"/>
    </xacro:sensor_asus_xtion_pro>

File: rb1_torso_description/urdf/rb1_torso_3dof.urdf.xacro (robot description, xacro)
@@ -6,4 +6,10 @@
   <xacro:property name="joint_damping" value="0.5"/>
   <xacro:property name="joint_friction" value="0.5"/>
+  <xacro:property name="j1_torso_mechanical_reduction" value="320.0"/>
+  <xacro:property name="j1_torso_motor_torque_constant" value="1.0"/>
+  <xacro:property name="j1_head_mechanical_reduction" value="320.0"/>
+  <xacro:property name="j1_head_motor_torque_constant" value="1.0"/>
+  <xacro:property name="j2_head_mechanical_reduction" value="320.0"/>
+  <xacro:property name="j2_head_motor_torque_constant" value="1.0"/>
   <xacro:macro name="rb1_torso_3dof" params="name hq">
   <!-- Robot mechanical and motor parameters -->
@@ -13,5 +19,5 @@
     name="base_link_rb1_torso">
   </link>
-  <link name="link1_rb1_torso">
+  <link name="link1_torso">
     <inertial>
       <mass value="3.0" />
@@ -51,9 +57,9 @@
       link="base_link_rb1_torso" />
     <child
-      link="link1_rb1_torso" />
+      link="link1_torso" />
     <axis
       xyz="0 0 0" />
   </joint>
-  <link name="link2_rb1_torso">
+  <link name="link2_torso">
     <inertial>
       <mass value="2.0" />
@@ -85,16 +91,25 @@
   </link>
   <joint
-	name="j1_rb1_torso"
+	name="j1_torso"
 	type="prismatic">
 	<origin
       xyz="0 0 0"
       rpy="0.0 0.0 0.0" />
-	<parent link="link1_rb1_torso" />
-    <child link="link2_rb1_torso" />
+	<parent link="link1_torso" />
+    <child link="link2_torso" />
     <axis xyz="0 0 1" />
     <limit effort="${joint_effort_limit}" velocity="${joint_velocity_limit}" upper="${0.360}" lower="${0}"/>
     <dynamics damping="${joint_damping}" friction="${joint_friction}"/>
   </joint>
-  <link name="link1_head_rb1_torso">
+  <transmission name="j1_torso_trans">
+	 <type>transmission_interface/SimpleTransmission</type>
+     <joint name="j1_torso" />
+     <actuator name="j1_torso_motor">
+	    <hardwareInterface>EffortJointInterface</hardwareInterface>
+        <mechanicalReduction>${j1_torso_mechanical_reduction}</mechanicalReduction>
+		<motorTorqueConstant>${j1_torso_motor_torque_constant}</motorTorqueConstant>
+	 </actuator>
+  </transmission>
+  <link name="link1_head">
     <inertial>
       <mass value="1.0" />
@@ -126,16 +141,25 @@
   </link>
   <joint
-	name="j1_head_rb1_torso"
+	name="j1_head"
 	type="revolute">
 	<origin
       xyz="0.010 0.0 0.940"
       rpy="0.0 0.0 0.0" />
-	<parent link="link2_rb1_torso" />
-    <child link="link1_head_rb1_torso" />
+	<parent link="link2_torso" />
+    <child link="link1_head" />
     <axis xyz="0 0 1" />
     <limit effort="${joint_effort_limit}" velocity="${joint_velocity_limit}" upper="${PI/2}" lower="${-PI/2}"/>
     <dynamics damping="${joint_damping}" friction="${joint_friction}"/>
   </joint>
-  <link name="link2_head_rb1_torso">
+  <transmission name="j1_head_trans">
+	 <type>transmission_interface/SimpleTransmission</type>
+     <joint name="j1_head" />
+     <actuator name="j1_head_motor">
+	    <hardwareInterface>EffortJointInterface</hardwareInterface>
+        <mechanicalReduction>${j1_head_mechanical_reduction}</mechanicalReduction>
+		<motorTorqueConstant>${j1_head_motor_torque_constant}</motorTorqueConstant>
+	 </actuator>
+  </transmission>
+  <link name="link2_head">
     <inertial>
       <mass value="1.0" />
@@ -167,15 +191,24 @@
   </link>
   <joint
-	name="j2_head_rb1_torso"
+	name="j2_head"
 	type="revolute">
 	<origin
       xyz="0.105 0.0 0.0"
       rpy="0.0 0.0 0.0" />
-	<parent link="link1_head_rb1_torso" />
-    <child link="link2_head_rb1_torso" />
+	<parent link="link1_head" />
+    <child link="link2_head" />
     <axis xyz="0 1 0" />
     <limit effort="${joint_effort_limit}" velocity="${joint_velocity_limit}" upper="${PI/4}" lower="${-PI/4}"/>
     <dynamics damping="${joint_damping}" friction="${joint_friction}"/>
   </joint>
+  <transmission name="j2_head_trans">
+	 <type>transmission_interface/SimpleTransmission</type>
+     <joint name="j2_head" />
+     <actuator name="j2_head_motor">
+	    <hardwareInterface>EffortJointInterface</hardwareInterface>
+        <mechanicalReduction>${j2_head_mechanical_reduction}</mechanicalReduction>
+		<motorTorqueConstant>${j2_head_motor_torque_constant}</motorTorqueConstant>
+	 </actuator>
+  </transmission>
   </xacro:macro>
 </robot>
