Commit message: Adding actual gripper v1 of the robot. Adding meshes, urdfs and updating simulation config files

File: rb1_arm_description/robots/rb1_arm.urdf (robot description, URDF)
Before this commit: robot rb1_arm, 7 links, 7 joints
Links:
- removed link link1_rb1_arm
- removed link motor1_rb1_arm
- added link end_effector_rb1_arm
- added link link01_rb1_arm, mass 0.506; collision mesh filename=package://rb1_arm_description/meshes/arms/armRB1_1_link.dae; visual mesh filename=package://rb1_arm_description/meshes/arms/armRB1_1_link.dae
- added link link34_rb1_arm, mass 0.351; collision mesh filename=package://rb1_arm_description/meshes/arms/armRB1_34_link.dae; visual mesh filename=package://rb1_arm_description/meshes/arms/armRB1_34_link.dae
- added link link45_rb1_arm, mass 0.388; collision mesh filename=package://rb1_arm_description/meshes/arms/armRB1_45_link.dae; visual mesh filename=package://rb1_arm_description/meshes/arms/armRB1_45_link.dae
- added link link56_rb1_arm, mass 0.3559; collision mesh filename=package://rb1_arm_description/meshes/arms/armRB1_56_link.dae; visual mesh filename=package://rb1_arm_description/meshes/arms/armRB1_56_link.dae
- added link link67_rb1_arm, mass 0.055; collision mesh filename=package://rb1_arm_description/meshes/arms/armRB1_67_link.dae; visual mesh filename=package://rb1_arm_description/meshes/arms/armRB1_67_link.dae
- added link motor01_rb1_arm, mass 0.855; collision mesh filename=package://rb1_arm_description/meshes/arms/armRB1_1_motor.dae; visual mesh filename=package://rb1_arm_description/meshes/arms/armRB1_1_motor.dae
- added link motor34_rb1_arm, mass 0.732; collision mesh filename=package://rb1_arm_description/meshes/arms/armRB1_34_motor.d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; visual mesh filename=package://rb1_arm_description/meshes/arms/armRB1_34_motor.d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
- added link motor45_rb1_arm, mass 0.732; collision mesh filename=package://rb1_arm_description/meshes/arms/armRB1_45_motor.d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; visual mesh filename=package://rb1_arm_description/meshes/arms/armRB1_45_motor.d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
- added link motor56_rb1_arm, mass 0.34; collision mesh filename=package://rb1_arm_description/meshes/arms/armRB1_56_motor.d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; visual mesh filename=package://rb1_arm_description/meshes/arms/armRB1_56_motor.d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
- added link motor67_rb1_arm, mass 0.34; collision mesh filename=package://rb1_arm_description/meshes/arms/armRB1_67_motor.d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; visual mesh filename=package://rb1_arm_description/meshes/arms/armRB1_67_motor.d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
- added link world
- link link12_rb1_arm: mass 1.0 -> 0.7
- link link23_rb1_arm: mass 1.0 -> 0.429
- link motor12_rb1_arm: mass 1.0 -> 0.855
- link motor23_rb1_arm: mass 1.0 -> 0.732
Joints:
- removed joint j12_rb1_arm
- removed joint j1m_rb1_arm
- removed joint j23_rb1_arm
- added joint fwf: type fixed, parent world, child base_link_rb1_arm
- added joint j01m_rb1_arm: type fixed, parent link01_rb1_arm, child motor01_rb1_arm, origin xyz=0.0 0.0 0.0 rpy=0.0 0.0 0.0, axis 0 0 0
- added joint j2: type revolute, parent link12_rb1_arm, child link23_rb1_arm, origin xyz=0.135 0 0 rpy=1.57079632679 0.0 0.0, axis 0 0 -1, limit lower=-1.570796327 upper=1.570796327 effort=60.0 velocity=2.9217
- added joint j3: type revolute, parent link23_rb1_arm, child link34_rb1_arm, origin xyz=0.310 0 0 rpy=0.0 0.0 0.0, axis 1 0 0, limit lower=-3.13 upper=3.13 effort=35.0 velocity=3.1527
- added joint j34m_rb1_arm: type fixed, parent link34_rb1_arm, child motor34_rb1_arm, origin xyz=0.0 0.0 0.0 rpy=0.0 0.0 0.0, axis 0 0 0
- added joint j4: type revolute, parent link34_rb1_arm, child link45_rb1_arm, origin xyz=0 0 0 rpy=0.0 0.0 0.0, axis 0 0 -1, limit lower=-1.570796327 upper=1.570796327 effort=35.0 velocity=3.1527
- added joint j45m_rb1_arm: type fixed, parent link45_rb1_arm, child motor45_rb1_arm, origin xyz=0.0 0.0 0.0 rpy=0.0 0.0 0.0, axis 0 0 0
- added joint j5: type revolute, parent link45_rb1_arm, child link56_rb1_arm, origin xyz=0.285 0 0 rpy=0.0 0.0 0.0, axis 1 0 0, limit lower=-3.13 upper=3.13 effort=35.0 velocity=3.1527
- added joint j56m_rb1_arm: type fixed, parent link56_rb1_arm, child motor56_rb1_arm, origin xyz=0.0 0.0 0.0 rpy=0.0 0.0 0.0, axis 0 0 0
- added joint j6: type revolute, parent link56_rb1_arm, child link67_rb1_arm, origin xyz=0 0 0 rpy=0.0 0.0 0.0, axis 0 0 -1, limit lower=-1.570796327 upper=1.570796327 effort=8.0 velocity=2.98452
- added joint j67m_rb1_arm: type fixed, parent link67_rb1_arm, child motor67_rb1_arm, origin xyz=0.0 0.0 0.0 rpy=0.0 0.0 0.0, axis 0 0 0
- added joint j7: type revolute, parent link67_rb1_arm, child end_effector_rb1_arm, origin xyz=0 0 0 rpy=0.0 0.0 0.0, axis 0 0 -1, limit lower=-3.13 upper=3.13 effort=8.0 velocity=2.98452
- joint j1: limit lower=-2.96706 upper=2.96706 effort=100.0 velocity=3.0 -> lower=-1.570796327 upper=1.570796327 effort=60.0 velocity=2.9217; origin xyz=0 0 0.19178 rpy=0.0 0.0 0.0 -> xyz=0 0 0 rpy=0.0 0.0 0.0; parent link1_rb1_arm -> link01_rb1_arm
- joint j1_rb1_arm: child link1_rb1_arm -> link01_rb1_arm

File: rb1_arm_description/robots/rb1_arm.urdf.xacro (robot description, xacro)
@@ -9,18 +9,15 @@
 	<!-- Import all available sensors -->
 	<!-- xacro:include filename="$(find rb1_arm_description)/urdf/sensors/all_sensors.urdf.xacro" / -->
-	<xacro:include filename="$(find rb1_arm_description)/urdf/grippers/two_finger_gripper.urdf.xacro" />
+	<xacro:include filename="$(find rb1_arm_description)/urdf/grippers/rb1_gripper_1.urdf.xacro" />
 	<!-- Joint elements -->
 	<joint
 	  name="gripper_joint"
       type="fixed">
-    <origin
-      xyz="0.0 0.0 0.0"
-      rpy="0.0 ${-PI/2} 0.0" />
-    <parent
-      link="end_effector_rb1_arm" />
-    <child
-      link="base_link_gripper" />
-    <axis
-      xyz="0 0 1" />
+		<origin
+		  xyz="0.055 0.0 0.0"
+		  rpy="0.0 0.0 0.0" />
+		<parent link="end_effector_rb1_arm" />
+		<child link="base_link_gripper" />
+		<axis xyz="1 0 0" />
 	</joint>
 	<!-- ***************** -->

File: rb1_arm_description/robots/rb1_arm_standalone.urdf.xacro (robot description, xacro)
@@ -13,19 +13,15 @@
 	<!-- Import RB1 arm elements -->
 	<xacro:include filename="$(find rb1_arm_description)/urdf/arms/rb1_arm_7dof.urdf.xacro" />
-	<xacro:include filename="$(find rb1_arm_description)/urdf/arms/rb1_arm_7dof.gazebo.xacro" />
-	<xacro:include filename="$(find rb1_arm_description)/urdf/grippers/two_finger_gripper.urdf.xacro" />
+	<xacro:include filename="$(find rb1_arm_description)/urdf/grippers/rb1_gripper_1.urdf.xacro" />
 	<!-- Joint elements -->
 	<joint
 	  name="gripper_joint"
       type="fixed">
-    <origin
-      xyz="0.0 0.0 0.0"
-      rpy="0.0 ${-PI/2} 0.0" />
-    <parent
-      link="end_effector_rb1_arm" />
-    <child
-      link="base_link_gripper" />
-    <axis
-      xyz="0 0 1" />
+		<origin
+		  xyz="0.055 0.0 0.0"
+		  rpy="0.0 0.0 0.0" />
+		<parent link="end_effector_rb1_arm" />
+		<child link="base_link_gripper" />
+		<axis xyz="1 0 0" />
 	</joint>
 	<!-- Import all available sensors -->

File: rb1_arm_description/urdf/arms/rb1_arm_7dof.gazebo.xacro (robot description, xacro)
@@ -3,48 +3,76 @@
   <!-- ros control plugin -->
   <xacro:macro name="ros_control">
-    <gazebo>
-      <plugin name="ros_control" filename="libgazebo_ros_control.so">
-        <robotNamespace>/rb1</robotNamespace>
-        <robotParam>robot_description</robotParam>
-        <controlPeriod>0.001</controlPeriod>
-	    <robotSimType>gazebo_ros_control/DefaultRobotHWSim</robotSimType>
-      </plugin>
-    </gazebo>
+	<gazebo>
+	  <plugin name="ros_control" filename="libgazebo_ros_control.so">
+		<robotNamespace>/rb1</robotNamespace>
+		<robotParam>robot_description</robotParam>
+		<controlPeriod>0.001</controlPeriod>
+		<robotSimType>gazebo_ros_control/DefaultRobotHWSim</robotSimType>
+	  </plugin>
+	</gazebo>
+   </xacro:macro>
 	<gazebo reference="base_link_rb1_arm">
 		<material>Gazebo/FlatBlack</material>
-		<turnGravityOff>true</turnGravityOff>
+		<turnGravityOff>false</turnGravityOff>
 	</gazebo>
 	<gazebo reference="link01_rb1_arm">
 		<material>Gazebo/Gray</material>
-		<turnGravityOff>true</turnGravityOff>
+		<turnGravityOff>false</turnGravityOff>
 	</gazebo>
 	<gazebo reference="motor01_rb1_arm">
 		<material>Gazebo/Black</material>
-		<turnGravityOff>true</turnGravityOff>
+		<turnGravityOff>false</turnGravityOff>
 	</gazebo>
 	<gazebo reference="link12_rb1_arm">
 		<material>Gazebo/Gray</material>
-		<turnGravityOff>true</turnGravityOff>
+		<turnGravityOff>false</turnGravityOff>
 	</gazebo>
 	<gazebo reference="motor12_rb1_arm">
 		<material>Gazebo/Black</material>
-		<turnGravityOff>true</turnGravityOff>
+		<turnGravityOff>false</turnGravityOff>
 	</gazebo>
 	<gazebo reference="link23_rb1_arm">
 		<material>Gazebo/Gray</material>
-		<turnGravityOff>true</turnGravityOff>
+		<turnGravityOff>false</turnGravityOff>
 	</gazebo>
 	<gazebo reference="motor23_rb1_arm">
 		<material>Gazebo/Black</material>
-		<turnGravityOff>true</turnGravityOff>
+		<turnGravityOff>false</turnGravityOff>
 	</gazebo>
 	<gazebo reference="link34_rb1_arm">
 		<material>Gazebo/Gray</material>
-		<turnGravityOff>true</turnGravityOff>
+		<turnGravityOff>false</turnGravityOff>
 	</gazebo>
 	<gazebo reference="motor34_rb1_arm">
 		<material>Gazebo/Black</material>
-		<turnGravityOff>true</turnGravityOff>
+		<turnGravityOff>false</turnGravityOff>
 	</gazebo>
-  </xacro:macro>
+	<gazebo reference="link45_rb1_arm">
+		<material>Gazebo/Gray</material>
+		<turnGravityOff>false</turnGravityOff>
+	</gazebo>
+	<gazebo reference="motor45_rb1_arm">
+		<material>Gazebo/Black</material>
+		<turnGravityOff>false</turnGravityOff>
+	</gazebo>
+	<gazebo reference="link56_rb1_arm">
+		<material>Gazebo/Gray</material>
+		<turnGravityOff>false</turnGravityOff>
+	</gazebo>
+	<gazebo reference="motor56_rb1_arm">
+		<material>Gazebo/Black</material>
+		<turnGravityOff>false</turnGravityOff>
+	</gazebo>
+	<gazebo reference="link67_rb1_arm">
+		<material>Gazebo/Gray</material>
+		<turnGravityOff>false</turnGravityOff>
+	</gazebo>
+	<gazebo reference="motor67_rb1_arm">
+		<material>Gazebo/Black</material>
+		<turnGravityOff>false</turnGravityOff>
+	</gazebo>
+    <gazebo reference="end_effector_rb1_arm">
+		<material>Gazebo/Gray</material>
+		<turnGravityOff>false</turnGravityOff>
+	</gazebo>
 </robot>

File: rb1_arm_description/urdf/arms/rb1_arm_7dof.urdf.xacro (robot description, xacro)
@@ -1,5 +1,5 @@
 <?xml version="1.0"?>
 <robot name="rb1_arm_7dof" xmlns:xacro="http://www.ros.org/wiki/xacro">
-  <!-- xacro:include filename="$(find rb1_arm_description)/urdf/arms/rb1_arm_7dof.gazebo.xacro" / -->
+	<xacro:include filename="$(find rb1_arm_description)/urdf/arms/rb1_arm_7dof.gazebo.xacro" />
 	<xacro:property name="j1_mechanical_reduction" value="502.0"/>
 	<xacro:property name="j1_motor_torque_constant" value="50.0"/>
@@ -690,48 +690,26 @@
 	 </actuator>
     </transmission>
-    <link name="end_effector_rb1_arm">
-	    <visual>
-		  <origin xyz="0 0 0.030" rpy="0 0 0" />
-		  <geometry>
-			<cylinder length="0.010" radius="0.015"/>
-		  </geometry>
-		</visual>
-		<collision>
-		  <origin xyz="0 0 0" rpy="0 0 0" />
-		  <geometry>
-			<cylinder length="0.005" radius="0.025"/>
-		  </geometry>
-		</collision>
-		<inertial>
-		  <origin xyz="0 0 0" rpy="0 0 0" />
-		  <mass value="0.1" />
-			<inertia
-			  ixx="0.01" ixy="0.0" ixz="0.0"
-			  iyy="0.01" iyz="0.0"
-			  izz="0.01" />
-		</inertial>
-    </link>
 	<!-- JOINT 7 -->
-	<joint
-		name="j7"
-		type="revolute">
+	<joint name="j7" type="revolute">
 	  <origin
         xyz="0 0 0"
-        rpy="0.0 ${PI/2} 0.0" />
+        rpy="0.0 0.0 0.0" />
 	  <parent link="link67_rb1_arm" />
       <child link="end_effector_rb1_arm" />
-      <axis xyz="0 0 -1" />
+      <axis xyz="1 0 0" />
       <limit effort="${joint_effort_limit_L42}" velocity="${joint_velocity_limit_L42}" upper="${j7_upper_limit}" lower="${j7_lower_limit}"/>
       <dynamics damping="${joint_damping}" friction="${joint_friction}"/>
     </joint>
     <transmission name="j7_trans">
-	 <type>transmission_interface/SimpleTransmission</type>
-     <joint name="j7" />
-     <actuator name="j7_motor">
-	    <hardwareInterface>EffortJointInterface</hardwareInterface>
-        <mechanicalReduction>${j7_mechanical_reduction}</mechanicalReduction>
-		<motorTorqueConstant>${j7_motor_torque_constant}</motorTorqueConstant>
-	 </actuator>
+		<type>transmission_interface/SimpleTransmission</type>
+		<joint name="j7" />
+		<actuator name="j7_motor">
+			<hardwareInterface>EffortJointInterface</hardwareInterface>
+			<mechanicalReduction>${j7_mechanical_reduction}</mechanicalReduction>
+			<motorTorqueConstant>${j7_motor_torque_constant}</motorTorqueConstant>
+		</actuator>
     </transmission>
+	<link name="end_effector_rb1_arm">
+    </link>
   </xacro:macro>
 </robot>

File: rb1_arm_description/urdf/grippers/rb1_gripper_1.urdf.xacro (robot description, xacro)
@@ -5,7 +5,7 @@
   <xacro:property name="joint_effort_limit" value="3.0"/>
   <xacro:property name="joint_velocity_limit" value="2.98452"/>
-	<xacro:property name="finger_lower_limit" value="-0.5"/>
-	<xacro:property name="finger_upper_limit" value="0.5"/>
-  <xacro:include filename="$(find rb1_arm_description)/urdf/grippers/two_finger_gripper.gazebo.xacro" />
+	<xacro:property name="finger_lower_limit" value="-0.7"/>
+	<xacro:property name="finger_upper_limit" value="0.0"/>
+  <xacro:include filename="$(find rb1_arm_description)/urdf/grippers/rb1_gripper_1.gazebo.xacro" />
   <link
     name="base_link_gripper">
@@ -15,12 +15,12 @@
         rpy="0 0 0" />
       <mass
-        value="0.2735" />
+        value="0.257" />
       <inertia
-        ixx="0.2735"
+        ixx="0.000131356"
         ixy="0.0"
-        ixz="0.0"
-        iyy="0.2735"
+        ixz="0.000000083"
+        iyy="0.000130775"
         iyz="0.0"
-        izz="0.2735" />
+        izz="0.00006918" />
     </inertial>
     <visual>
@@ -30,5 +30,5 @@
       <geometry>
         <mesh
-          filename="package://rb1_arm_description/meshes/grippers/base_gripper.dae" />
+          filename="package://rb1_arm_description/meshes/grippers/v1/gripper_motor.dae" />
       </geometry>
       <material
@@ -44,5 +44,5 @@
       <geometry>
         <mesh
-          filename="package://rb1_arm_description/meshes/grippers/base_gripper.dae" />
+          filename="package://rb1_arm_description/meshes/grippers/v1/gripper_motor.dae" />
       </geometry>
       <contact_coefficients kd="1.0" kp="1000.0" mu="0"/>
@@ -56,12 +56,12 @@
         rpy="0 0 0" />
       <mass
-        value="0.03" />
+        value="0.1264" />
       <inertia
-        ixx="0.03"
-        ixy="0.0"
-        ixz="0.0"
-        iyy="0.03"
-        iyz="0.0"
-        izz="0.03" />
+        ixx="0.000097351"
+        ixy="0.000056737"
+        ixz="0.000000245"
+        iyy="0.000315015"
+        iyz="0.000001224"
+        izz="0.000319853" />
     </inertial>
     <visual>
@@ -71,5 +71,5 @@
       <geometry>
         <mesh
-          filename="package://rb1_arm_description/meshes/grippers/finger1.dae" />
+          filename="package://rb1_arm_description/meshes/grippers/v1/gripper_link1.dae" />
       </geometry>
       <material
@@ -85,5 +85,5 @@
       <geometry>
         <mesh
-          filename="package://rb1_arm_description/meshes/grippers/finger1.dae" />
+          filename="package://rb1_arm_description/meshes/grippers/v1/gripper_link1.dae" />
       </geometry>
     </collision>
@@ -91,26 +91,13 @@
   <joint
     name="jg1"
-    type="revolute">
+    type="fixed">
     <origin
-      xyz="0.097993 0.028575 0"
-      rpy="3.0028E-16 5.9154E-22 2.2204E-16" />
+      xyz="0.0 0.0 0"
+      rpy="0.0 0.0 0.0" />
     <parent
       link="base_link_gripper" />
     <child
       link="link_finger1" />
-    <axis
-      xyz="0 0 -1" />
-    <limit effort="${joint_effort_limit}" velocity="${joint_velocity_limit}" upper="${finger_upper_limit}" lower="${finger_lower_limit}"/>
-    <dynamics damping="${joint_damping}" friction="${joint_friction}"/>
   </joint>
-  <transmission name="jg1_trans">
-	 <type>transmission_interface/SimpleTransmission</type>
-     <joint name="jg1" />
-     <actuator name="jg1_motor">
-	    <hardwareInterface>EffortJointInterface</hardwareInterface>
-        <mechanicalReduction>${finger_mechanical_reduction}</mechanicalReduction>
-		<motorTorqueConstant>${finger_motor_torque_constant}</motorTorqueConstant>
-	 </actuator>
-  </transmission>
   <link
     name="link_finger2">
@@ -120,12 +107,12 @@
         rpy="0 0 0" />
       <mass
-        value="0.03" />
+        value="0.0633" />
       <inertia
-        ixx="0.03"
-        ixy="0.0"
-        ixz="0.0"
-        iyy="0.03"
-        iyz="0.0"
-        izz="0.03" />
+        ixx="0.000062574"
+        ixy="-0.00005905"
+        ixz="0.000009803"
+        iyy="0.000292473"
+        iyz="-0.00000366"
+        izz="0.00027232" />
     </inertial>
     <visual>
@@ -135,5 +122,5 @@
       <geometry>
         <mesh
-          filename="package://rb1_arm_description/meshes/grippers/finger2.dae" />
+          filename="package://rb1_arm_description/meshes/grippers/v1/gripper_link2.dae" />
       </geometry>
       <material
@@ -149,5 +136,5 @@
       <geometry>
         <mesh
-          filename="package://rb1_arm_description/meshes/grippers/finger2.dae" />
+          filename="package://rb1_arm_description/meshes/grippers/v1/gripper_link1.dae" />
       </geometry>
     </collision>
@@ -157,6 +144,6 @@
     type="revolute">
     <origin
-      xyz="0.097993 -0.028575 0"
-      rpy="3.0028E-16 7.477E-22 -5.1764E-15" />
+      xyz="0.0 0.0 0"
+      rpy="0.0 0.0 0.0" />
     <parent
       link="base_link_gripper" />
@@ -177,14 +164,3 @@
 	 </actuator>
   </transmission>
-  <!-- Grasp link GRIPPER  -->
-	<link name="gripper_grasp_link1">
-	</link>
-	<joint name="gripper_grasp_joint1" type="fixed">
-		<origin xyz="0.14 0 0" rpy="0.0 0.0 0.0" />
-		<parent link="base_link_gripper"/>
-		<child link="gripper_grasp_link1"/>
-	</joint>
-  <!-- TCP management -->
-  <!-- Import all Gazebo-customization elements, including Gazebo colors -->
-  <!-- xacro:include filename="$(find rb1_arm_description)/urdf/tcp.urdf.xacro" / -->
 </robot>
