Commit message: rb1_base_ description, control, gazebo adapted files for standalone sim and in robot

File: rb1_base_description/robots/rb1_base_platform_standalone.urdf.xacro (robot description, xacro)
@@ -7,4 +7,12 @@
 	<!-- Import RB1 base elements -->
     <xacro:include filename="$(find rb1_base_description)/urdf/bases/rb1_base.urdf.xacro" />
+    <gazebo>
+      <plugin name="ros_control" filename="libgazebo_ros_control.so">
+        <robotNamespace>/rb1</robotNamespace>
+        <robotParam>robot_description</robotParam>
+        <controlPeriod>0.001</controlPeriod>
+	    <robotSimType>gazebo_ros_control/DefaultRobotHWSim</robotSimType>
+      </plugin>
+    </gazebo>
 	<!-- Import RB1 wheels -->
 	<xacro:include filename="$(find rb1_base_description)/urdf/wheels/rubber_wheel.urdf.xacro" />

File: rb1_base_description/urdf/bases/rb1_base.gazebo.xacro (robot description, xacro)
@@ -2,14 +2,14 @@
 <robot xmlns:xacro="http://ros.org/wiki/xacro">
   <!-- ros control plugin -->
-  <xacro:macro name="ros_control">
+  <!-- xacro:macro name="ros_control">
     <gazebo>
       <plugin name="ros_control" filename="libgazebo_ros_control.so">
-        <robotNamespace>/rb1_base</robotNamespace>
+        <robotNamespace>/rb1</robotNamespace>
         <robotParam>robot_description</robotParam>
-        <controlPeriod>0.001</controlPeriod> <!-- controlPeriod>0.003</controlPeriod -->
+        <controlPeriod>0.001</controlPeriod>
 	    <robotSimType>gazebo_ros_control/DefaultRobotHWSim</robotSimType>
       </plugin>
     </gazebo>
-	</xacro:macro>
+	</xacro:macro -->
 	<!-- differential drive plugin -->
 	<xacro:macro name="diff_drive">
