Commit message: castor wheels are fixed, with no friction, corrected collision dimensions

File: rb1_base_description/robots/rb1_base_platform.urdf.xacro (robot description, xacro)
@@ -23,8 +23,10 @@
 	<xacro:property name="omni_back_x" value="0.185" />
 	<xacro:property name="omni_back_y" value="0.0" />
-	<xacro:property name="omni_back_z" value="0.026" />
+	<!-- xacro:property name="omni_back_z" value="0.028" / -->
+	<xacro:property name="omni_back_z" value="0.030" />
 	<xacro:property name="omni_front_x" value="0.133" />
 	<xacro:property name="omni_front_y" value="0.142" />
-	<xacro:property name="omni_front_z" value="0.026" />
+	<!-- xacro:property name="omni_front_z" value="0.028" / -->
+	<xacro:property name="omni_front_z" value="0.030" />
 	<!-- Flag to select the high or low quality model -->
 	<xacro:property name="hq" value="true" />
@@ -35,7 +37,7 @@
 	<!-- RB-1 base -->
 	<xacro:rb1_base name="rb1_base" publish_bf="true" hq="${hq}" />
-	<!-- Gazebo ros control pluggins -->
+	<!-- Gazebo ros control plugins -->
 	<xacro:ros_control/>
-	<!-- Gazebo skid steering pluggins -->
+	<!-- Gazebo skid steering plugins -->
 	<xacro:diff_drive/>
 	<!-- WHEELS -->
@@ -49,4 +51,10 @@
 	<xacro:omni_wheel name="omni_back" parent="base_link" hq="${hq}">
 		<origin xyz="-${omni_back_x} ${omni_back_y} ${omni_back_z}" rpy="0 0 0"/>
+	</xacro:omni_wheel>
+	<xacro:omni_wheel name="omni_front_left" parent="base_link" hq="${hq}">
+		<origin xyz="${omni_front_x} ${omni_front_y} ${omni_front_z}" rpy="0 0 0"/>
+	</xacro:omni_wheel>
+	<xacro:omni_wheel name="omni_front_right" parent="base_link" hq="${hq}">
+		<origin xyz="${omni_front_x} -${omni_front_y} ${omni_front_z}" rpy="0 0 0"/>
 	</xacro:omni_wheel>
 	<!-- SENSORS -->

File: rb1_base_description/urdf/bases/rb1_base.gazebo.xacro (robot description, xacro)
@@ -22,5 +22,5 @@
         <wheelSeparation>0.5380</wheelSeparation>
         <wheelDiameter>0.2410</wheelDiameter>
-        <torque>20</torque>
+        <!-- torque>20</torque -->
         <commandTopic>cmd_vel</commandTopic>
         <odometryTopic>odom</odometryTopic>
@@ -28,5 +28,12 @@
         <robotBaseFrame>base_footprint</robotBaseFrame>
         <robotNamespace>/rb1_base</robotNamespace>
-        <!-- broadcastTF>1</broadcastTF -->
+        <rosDebugLevel>na</rosDebugLevel>
+        <publishWheelTF>false</publishWheelTF>
+        <publishWheelJointState>false</publishWheelJointState>
+        <wheelAcceleration>0</wheelAcceleration>
+        <wheelTorque>5</wheelTorque>
+        <!-- odometrySource>"encoder"</odometrySource -->
+        <odometrySource>"world"</odometrySource>
+        <publishTf>0.0000</publishTf>
 	</plugin>
 	</gazebo>

File: rb1_base_description/urdf/bases/rb1_base.urdf.xacro (robot description, xacro)
@@ -17,5 +17,7 @@
     </link>
     <joint name="base_footprint_joint" type="fixed">
-      <origin xyz="0 0 ${wheel_radius}" rpy="0 0 0" /> <!-- ${wheel_radius} property must be defined inside wheel description -->
+      <!-- origin xyz="0 0 ${wheel_radius}" rpy="0 0 0" / -->
+       <!-- origin xyz="0 0 ${wheel_radius - wheel_offset_z}" rpy="0 0 0" / -->
+       <origin xyz="0 0 0.025" rpy="0 0 0" />
       <parent link="base_footprint"/>
       <child link="base_link" />
@@ -36,19 +38,19 @@
        </geometry>
        </xacro:if>
-       <!-- xacro:unless value="${hq}">
+       <xacro:unless value="${hq}">
        <geometry>
-       <mesh filename="package://rb1_base_description/meshes/bases/rb1_base_simple.stl"/>
+       <mesh filename="package://rb1_base_description/meshes/bases/rb1_base.stl"/>
        </geometry>
-       </xacro:unless -->
+       </xacro:unless>
        <material name="darkgrey">
          <color rgba="0.1 0.1 0.1 1"/>
        </material>
     </visual>
-    <collision>
+    <!-- collision>
        <origin xyz="0 0 0" rpy="0 0 0 " />
        <geometry>
          <mesh filename="package://rb1_base_description/meshes/bases/rb1_base.dae"/>
        </geometry>
-    </collision>
+    </collision -->
   </link>
   </xacro:macro>

File: rb1_base_description/urdf/wheels/omni_wheel.urdf.xacro (robot description, xacro)
@@ -3,15 +3,16 @@
   <xacro:property name="M_PI" value="3.1415926535897931" />
   <!-- Wheels -->
-  <property name="wheel_radius" value="0.076" />
-  <property name="wheel_height" value="0.050" />
-  <property name="wheel_mass" value="1.0" /> <!-- in kg-->
+  <property name="omni_wheel_radius" value="0.051" />
+  <property name="omni_wheel_height" value="0.025" />
+  <property name="omni_wheel_mass" value="0.3" /> <!-- in kg-->
   <xacro:macro name="cylinder_inertia" params="m r h">
     <inertia  ixx="${m*(3*r*r+h*h)/12}" ixy = "0" ixz = "0"
               iyy="${m*(3*r*r+h*h)/12}" iyz = "0"
               izz="${m*r*r/2}" />
-  </xacro:macro>interc
+  </xacro:macro>
   <xacro:macro name="omni_wheel" params="name parent *origin hq">
 <!--WHEEL TIRE -->
-    <joint name="joint_${name}_wheel" type="continuous">
+    <!-- joint name="joint_${name}_wheel" type="continuous" -->
+    <joint name="joint_${name}_wheel" type="fixed">
       <parent link="${parent}"/>
       <child link="${name}_wheel"/>
@@ -34,5 +35,5 @@
           <origin xyz="0 0 0" rpy="${M_PI/2} 0 0" />
           <geometry>
-            <cylinder length="${wheel_height}" radius="${wheel_radius}" />
+            <cylinder length="${omni_wheel_height}" radius="${omni_wheel_radius}" />
           </geometry>
         </xacro:unless>
@@ -41,5 +42,5 @@
       <origin xyz="0 0 0" rpy="${M_PI/2} 0 0" />
         <geometry>
-          <cylinder length="${wheel_height}" radius="${wheel_radius}" />
+          <cylinder length="${omni_wheel_height}" radius="${omni_wheel_radius}" />
         </geometry>
       </collision>
@@ -53,9 +54,9 @@
         <mass value="${wheel_mass}" />
         <origin xyz="0 0 0" />
-        <cylinder_inertia  m="${wheel_mass}" r="${wheel_radius}" h="${wheel_height}" />
+        <cylinder_inertia  m="${omni_wheel_mass}" r="${omni_wheel_radius}" h="${omni_wheel_height}" />
         <!-- inertia  ixx="0.001" ixy="0.0"  ixz="0.0"  iyy="0.001"  iyz="0.0"  izz="0.001" / -->
       </inertial>
     </link>
-    <transmission name="${name}_wheel_joint_trans">
+    <!-- transmission name="${name}_wheel_joint_trans">
       <type>transmission_interface/SimpleTransmission</type>
       <joint name="joint_${name}_wheel" />
@@ -64,8 +65,6 @@
         <mechanicalReduction>1</mechanicalReduction>
       </actuator>
-    </transmission>
+    </transmission -->
     <gazebo reference="${name}_wheel">
-			<!-- mu1 value="5.0"/>
-			<mu2 value="0.5"/ -->
 			<mu1 value="0.0"/>
 			<mu2 value="0.0"/>
@@ -73,5 +72,5 @@
 			<kd value="1.0" />
 			<fdir1 value="1 0 0"/>
-      <turnGravityOff>false</turnGravityOff>
+            <turnGravityOff>false</turnGravityOff>
     </gazebo>
   </xacro:macro>

File: rb1_base_description/urdf/wheels/rubber_wheel.urdf.xacro (robot description, xacro)
@@ -44,5 +44,5 @@
       </visual>
       <collision>
-				<origin xyz="0 0 0" rpy="${M_PI/2} 0 0" />
+		<origin xyz="0 0 0" rpy="${M_PI/2} 0 0" />
         <geometry>
           <cylinder length="${wheel_height}" radius="${wheel_radius}" />

Commit message: added laser sensors, corrected bug in number of rays urg04, diff_drive plugin left by right

File: rb1_base_description/robots/rb1_base_platform.urdf.xacro (robot description, xacro)
@@ -62,9 +62,7 @@
 		<origin xyz="0.0 0.0 0.33" rpy="0 0 0"/>
 	</xacro:sensor_hokuyo_utm30lx>
-<!--
     <xacro:sensor_hokuyo_urg04lx name="hokuyo1" parent="base_link">
-        <origin xyz="-0.1 0.0 0.33" rpy="0 0 0"/>
+        <origin xyz="0.220 0.0 0.170" rpy="0 3.1416 3.1416"/>
     </xacro:sensor_hokuyo_urg04lx>
--->
 	<xacro:sensor_imu name="imu" parent="base_link">
 		<origin xyz="-0.18 0.0 0.170" rpy="0 0 0"/>

File: rb1_base_description/urdf/bases/rb1_base.gazebo.xacro (robot description, xacro)
@@ -18,14 +18,15 @@
 	    <alwaysOn>true</alwaysOn>
         <updateRate>50.0</updateRate>
-        <leftJoint>joint_left_wheel</leftJoint>
-        <rightJoint>joint_right_wheel</rightJoint>
-        <wheelSeparation>0.5380</wheelSeparation>
-        <wheelDiameter>0.2410</wheelDiameter>
-        <!-- torque>20</torque -->
+        <!-- leftJoint>joint_left_wheel</leftJoint>
+        <rightJoint>joint_right_wheel</rightJoint -->
+        <leftJoint>joint_right_wheel</leftJoint>
+        <rightJoint>joint_left_wheel</rightJoint>
+        <wheelSeparation>0.3660</wheelSeparation>
+        <wheelDiameter>0.1524</wheelDiameter>
         <commandTopic>cmd_vel</commandTopic>
         <odometryTopic>odom</odometryTopic>
         <odometryFrame>odom</odometryFrame>
         <robotBaseFrame>base_footprint</robotBaseFrame>
-        <robotNamespace>/rb1_base</robotNamespace>
+        <!-- robotNamespace></robotNamespace -->
         <rosDebugLevel>na</rosDebugLevel>
         <publishWheelTF>false</publishWheelTF>
@@ -33,7 +34,7 @@
         <wheelAcceleration>0</wheelAcceleration>
         <wheelTorque>5</wheelTorque>
-        <!-- odometrySource>"encoder"</odometrySource -->
-        <odometrySource>"world"</odometrySource>
-        <publishTf>0.0000</publishTf>
+        <odometrySource>encoder</odometrySource>
+        <!-- odometrySource>world</odometrySource -->
+        <publishTf>1</publishTf>
 	</plugin>
 	</gazebo>

File: rb1_base_description/urdf/sensors/hokuyo_urg04lx.urdf.xacro (robot description, xacro)
@@ -41,6 +41,6 @@
 							<samples>681</samples>
 							<resolution>1</resolution>
-							<min_angle>2.0943951</min_angle>
-							<max_angle>-2.0943951</max_angle>
+							<min_angle>-2.0943951</min_angle>
+							<max_angle>2.0943951</max_angle>
 						</horizontal>
 					</scan>

File: rb1_base_description/urdf/wheels/rubber_wheel.urdf.xacro (robot description, xacro)
@@ -55,5 +55,5 @@
       </inertial>
     </link>
-    <!-- Transmission is important to link the joints and the controller (see summit_xl_control/config/summit_xl_control.yaml)-->
+    <!-- Transmission is important to link the joints and the controller (see rb1_control/config/rb1_control.yaml)-->
     <transmission name="${name}_wheel_joint_trans">
       <type>transmission_interface/SimpleTransmission</type>

Commit message: changed castor collision to spheres, some positions adjustments

File: rb1_base_description/robots/rb1_base_platform.urdf.xacro (robot description, xacro)
@@ -24,9 +24,9 @@
 	<xacro:property name="omni_back_y" value="0.0" />
 	<!-- xacro:property name="omni_back_z" value="0.028" / -->
-	<xacro:property name="omni_back_z" value="0.030" />
+	<xacro:property name="omni_back_z" value="0.0265" />
 	<xacro:property name="omni_front_x" value="0.133" />
 	<xacro:property name="omni_front_y" value="0.142" />
 	<!-- xacro:property name="omni_front_z" value="0.028" / -->
-	<xacro:property name="omni_front_z" value="0.030" />
+	<xacro:property name="omni_front_z" value="0.0265" />
 	<!-- Flag to select the high or low quality model -->
 	<xacro:property name="hq" value="true" />
@@ -60,5 +60,5 @@
 	<!-- SENSORS -->
 	<xacro:sensor_hokuyo_utm30lx name="hokuyo" parent="base_link">
-		<origin xyz="0.0 0.0 0.33" rpy="0 0 0"/>
+		<origin xyz="0.210 0.0 0.305" rpy="0 0 0"/>
 	</xacro:sensor_hokuyo_utm30lx>
     <xacro:sensor_hokuyo_urg04lx name="hokuyo1" parent="base_link">

File: rb1_base_description/urdf/bases/rb1_base.urdf.xacro (robot description, xacro)
@@ -18,6 +18,6 @@
     <joint name="base_footprint_joint" type="fixed">
       <!-- origin xyz="0 0 ${wheel_radius}" rpy="0 0 0" / -->
-       <!-- origin xyz="0 0 ${wheel_radius - wheel_offset_z}" rpy="0 0 0" / -->
-       <origin xyz="0 0 0.025" rpy="0 0 0" />
+       <origin xyz="0 0 ${wheel_radius - wheel_offset_z}" rpy="0 0 0" />
+       <!-- origin xyz="0 0 0.025" rpy="0 0 0" / -->
       <parent link="base_footprint"/>
       <child link="base_link" />
@@ -47,10 +47,10 @@
        </material>
     </visual>
-    <!-- collision>
+    <collision>
        <origin xyz="0 0 0" rpy="0 0 0 " />
        <geometry>
          <mesh filename="package://rb1_base_description/meshes/bases/rb1_base.dae"/>
        </geometry>
-    </collision -->
+    </collision>
   </link>
   </xacro:macro>

File: rb1_base_description/urdf/wheels/omni_wheel.urdf.xacro (robot description, xacro)
@@ -39,16 +39,16 @@
         </xacro:unless>
       </visual>
-      <collision>
+      <!-- collision>
       <origin xyz="0 0 0" rpy="${M_PI/2} 0 0" />
         <geometry>
           <cylinder length="${omni_wheel_height}" radius="${omni_wheel_radius}" />
         </geometry>
-      </collision>
-      <!-- collision>
+      </collision -->
+      <collision>
       <origin xyz="0 0 0" rpy="${M_PI/2} 0 0" />
        <geometry>
-         <sphere radius="${wheel_radius}"/>
+         <sphere radius="${omni_wheel_radius}"/>
        </geometry>
-      </collision -->
+      </collision>
       <inertial>
         <mass value="${wheel_mass}" />

Commit message: rb1_base_description: Changing name of laser sensor

File: rb1_base_description/robots/rb1_base_platform.urdf.xacro (robot description, xacro)
@@ -59,10 +59,10 @@
 	</xacro:omni_wheel>
 	<!-- SENSORS -->
-	<xacro:sensor_hokuyo_utm30lx name="hokuyo" parent="base_link">
+	<!-- xacro:sensor_hokuyo_utm30lx name="hokuyo" parent="base_link">
 		<origin xyz="0.210 0.0 0.305" rpy="0 0 0"/>
-	</xacro:sensor_hokuyo_utm30lx>
-    <xacro:sensor_hokuyo_urg04lx name="hokuyo1" parent="base_link">
-        <origin xyz="0.220 0.0 0.170" rpy="0 3.1416 3.1416"/>
-    </xacro:sensor_hokuyo_urg04lx>
+	</xacro:sensor_hokuyo_utm30lx -->
+        <xacro:sensor_hokuyo_urg04lx name="hokuyo" parent="base_link">
+           <origin xyz="0.220 0.0 0.170" rpy="0 3.1416 3.1416"/>
+        </xacro:sensor_hokuyo_urg04lx>
 	<xacro:sensor_imu name="imu" parent="base_link">
 		<origin xyz="-0.18 0.0 0.170" rpy="0 0 0"/>
