Commit message: rb1_arm_(description,gazebo,control): Setting urdf inertial params for the arm, and configuring PID values for the arm and torso

File: rb1_arm_description/urdf/arms/rb1_arm_7dof.gazebo.xacro (robot description, xacro)
@@ -11,4 +11,40 @@
       </plugin>
     </gazebo>
+	<gazebo reference="base_link_rb1_arm">
+		<material>Gazebo/FlatBlack</material>
+		<turnGravityOff>true</turnGravityOff>
+	</gazebo>
+	<gazebo reference="link01_rb1_arm">
+		<material>Gazebo/Gray</material>
+		<turnGravityOff>true</turnGravityOff>
+	</gazebo>
+	<gazebo reference="motor01_rb1_arm">
+		<material>Gazebo/Black</material>
+		<turnGravityOff>true</turnGravityOff>
+	</gazebo>
+	<gazebo reference="link12_rb1_arm">
+		<material>Gazebo/Gray</material>
+		<turnGravityOff>true</turnGravityOff>
+	</gazebo>
+	<gazebo reference="motor12_rb1_arm">
+		<material>Gazebo/Black</material>
+		<turnGravityOff>true</turnGravityOff>
+	</gazebo>
+	<gazebo reference="link23_rb1_arm">
+		<material>Gazebo/Gray</material>
+		<turnGravityOff>true</turnGravityOff>
+	</gazebo>
+	<gazebo reference="motor23_rb1_arm">
+		<material>Gazebo/Black</material>
+		<turnGravityOff>true</turnGravityOff>
+	</gazebo>
+	<gazebo reference="link34_rb1_arm">
+		<material>Gazebo/Gray</material>
+		<turnGravityOff>true</turnGravityOff>
+	</gazebo>
+	<gazebo reference="motor34_rb1_arm">
+		<material>Gazebo/Black</material>
+		<turnGravityOff>true</turnGravityOff>
+	</gazebo>
   </xacro:macro>
 </robot>

File: rb1_arm_description/urdf/arms/rb1_arm_7dof.urdf.xacro (robot description, xacro)
@@ -2,24 +2,41 @@
 <robot name="rb1_arm_7dof" xmlns:xacro="http://www.ros.org/wiki/xacro">
   <!-- xacro:include filename="$(find rb1_arm_description)/urdf/arms/rb1_arm_7dof.gazebo.xacro" / -->
-  <xacro:include filename="$(find rb1_arm_description)/urdf/links/rb1_arm_link.urdf.xacro" />
-  <xacro:property name="j1_mechanical_reduction" value="502.0"/>
-  <xacro:property name="j1_motor_torque_constant" value="50.0"/>
-  <xacro:property name="j2_mechanical_reduction" value="502.0"/>
-  <xacro:property name="j2_motor_torque_constant" value="50.0"/>
-  <xacro:property name="j3_mechanical_reduction" value="502.0"/>
-  <xacro:property name="j3_motor_torque_constant" value="5.0"/>
-  <xacro:property name="j4_mechanical_reduction" value="502.0"/>
-  <xacro:property name="j4_motor_torque_constant" value="5.0"/>
-  <xacro:property name="j5_mechanical_reduction" value="502.0"/>
-  <xacro:property name="j5_motor_torque_constant" value="5.0"/>
-  <xacro:property name="j6_mechanical_reduction" value="304.0"/>
-  <xacro:property name="j6_motor_torque_constant" value="3.0"/>
-  <xacro:property name="j7_mechanical_reduction" value="304.0"/>
-  <xacro:property name="j7_motor_torque_constant" value="3.0"/>
-  <xacro:property name="joint_effort_limit" value="2500.0"/>
-  <xacro:property name="joint_velocity_limit" value="3.0"/>
-  <xacro:property name="joint_damping" value="0.1"/>
-  <xacro:property name="joint_friction" value="0.1"/>
-  <xacro:macro name="rb1_arm_7dof" params="name hq">
+	<xacro:property name="j1_mechanical_reduction" value="502.0"/>
+	<xacro:property name="j1_motor_torque_constant" value="50.0"/>
+	<xacro:property name="j2_mechanical_reduction" value="502.0"/>
+	<xacro:property name="j2_motor_torque_constant" value="50.0"/>
+	<xacro:property name="j3_mechanical_reduction" value="502.0"/>
+	<xacro:property name="j3_motor_torque_constant" value="50.0"/>
+	<xacro:property name="j4_mechanical_reduction" value="502.0"/>
+	<xacro:property name="j4_motor_torque_constant" value="5.0"/>
+	<xacro:property name="j5_mechanical_reduction" value="502.0"/>
+	<xacro:property name="j5_motor_torque_constant" value="5.0"/>
+	<xacro:property name="j6_mechanical_reduction" value="304.0"/>
+	<xacro:property name="j6_motor_torque_constant" value="3.0"/>
+	<xacro:property name="j7_mechanical_reduction" value="304.0"/>
+	<xacro:property name="j7_motor_torque_constant" value="3.0"/>
+	<xacro:property name="j1_lower_limit" value="-1.570796327"/>
+	<xacro:property name="j1_upper_limit" value="1.570796327"/>
+	<xacro:property name="j2_lower_limit" value="-1.570796327"/>
+	<xacro:property name="j2_upper_limit" value="1.570796327"/>
+	<xacro:property name="j3_lower_limit" value="-3.13"/>
+	<xacro:property name="j3_upper_limit" value="3.13"/>
+	<xacro:property name="j4_lower_limit" value="-1.570796327"/>
+	<xacro:property name="j4_upper_limit" value="1.570796327"/>
+	<xacro:property name="j5_lower_limit" value="-3.13"/>
+	<xacro:property name="j5_upper_limit" value="3.13"/>
+	<xacro:property name="j6_lower_limit" value="-1.570796327"/>
+	<xacro:property name="j6_upper_limit" value="1.570796327"/>
+	<xacro:property name="j7_lower_limit" value="-3.13"/>
+	<xacro:property name="j7_upper_limit" value="3.13"/>
+	<xacro:property name="joint_effort_limit_H54_200" value="60.0"/>
+	<xacro:property name="joint_velocity_limit_H54_200" value="2.9217"/>
+	<xacro:property name="joint_effort_limit_H54_100" value="35.0"/>
+	<xacro:property name="joint_velocity_limit_H54_100" value="3.1527"/>
+	<xacro:property name="joint_effort_limit_L42" value="8.0"/>
+	<xacro:property name="joint_velocity_limit_L42" value="2.98452"/>
+	<xacro:property name="joint_damping" value="0.7"/>
+	<xacro:property name="joint_friction" value="0.5"/>
+	<xacro:macro name="rb1_arm_7dof" params="name hq">
     <!-- Robot mechanical and motor parameters -->
     <xacro:property name="PI" value="3.1415926535897931"/>
@@ -28,36 +45,174 @@
       name="base_link_rb1_arm">
     </link>
-    <xacro:arm_link name="arm_link1" hq="${hq}" parent="" num="01"/>
-    <xacro:arm_link name="arm_link2" hq="${hq}" parent="" num="12"/>
-    <xacro:arm_link name="arm_link3" hq="${hq}" parent="" num="23"/>
-    <xacro:arm_link name="arm_link4" hq="${hq}" parent="" num="34"/>
-    <xacro:arm_link name="arm_link5" hq="${hq}" parent="" num="45"/>
-    <xacro:arm_link name="arm_link6" hq="${hq}" parent="" num="56"/>
-    <xacro:arm_link name="arm_link7" hq="${hq}" parent="" num="67"/>
-	<joint
-	  name="j1_rb1_arm"
-      type="fixed">
-    <origin
-      xyz="0.0 0.0 0.0"
-      rpy="0.0 0.0 0.0" />
-    <parent
-      link="base_link_rb1_arm" />
-    <child
-      link="link1_rb1_arm" />
-    <axis
-      xyz="0 0 0" />
+	<joint
+		  name="j1_rb1_arm"
+		  type="fixed">
+		<origin
+		  xyz="0.0 0.0 0.0"
+		  rpy="0.0 0.0 0.0" />
+		<parent
+		  link="base_link_rb1_arm" />
+		<child
+		  link="link01_rb1_arm" />
+		<axis
+		  xyz="0 0 0" />
+	</joint>
+	<!-- 01 -->
+	<link name="link01_rb1_arm">
+		<inertial>
+		  <mass value="0.506" />
+		  <origin xyz="-0.05161 0 -0.003" />
+		  <inertia  ixx="0.0014526484" ixy="0.0"  ixz="-8.792613e-005" iyy="0.0018217854" iyx="0.0"  iyz="0.0" izz="0.0008987159" />
+		</inertial>
+		<visual>
+		   <origin xyz="0 0 0" rpy="0 0 0" />
+		   <xacro:if value="${hq}">
+		   <geometry>
+			 <mesh filename="package://rb1_arm_description/meshes/arms/armRB1_1_link.dae"/>
+		   </geometry>
+		   </xacro:if>
+		   <xacro:unless value="${hq}">
+		   <geometry>
+		   <mesh filename="package://rb1_arm_description/meshes/arms/armRB1_1_link.stl"/>
+		   </geometry>
+		   </xacro:unless>
+		   <material name="darkgrey">
+			 <color rgba="0.1 0.1 0.1 1"/>
+		   </material>
+		</visual>
+		<collision>
+		   <origin xyz="0 0 0" rpy="0 0 0 " />
+		   <geometry>
+			 <mesh filename="package://rb1_arm_description/meshes/arms/armRB1_1_link.dae"/>
+		   </geometry>
+		</collision>
+	</link>
+	<link name="motor01_rb1_arm">
+		<inertial>
+		  <mass value="0.855" />
+		  <origin xyz="0 0 0.00693" />
+		  <!--inertia  ixx="0.01" ixy="0.0"  ixz="0.0"  iyy="0.01"  iyz="0.0"  izz="0.01" /-->
+		  <inertia ixx="0.001211476" ixy="0.0" ixz="6.05332e-006" iyy="0.001211334" iyz="0.0" izz="0.0003787678"/>
+		</inertial>
+		<visual>
+		   <origin xyz="0 0 0" rpy="0 0 0" />
+		   <xacro:if value="${hq}">
+		   <geometry>
+			 <mesh filename="package://rb1_arm_description/meshes/arms/armRB1_1_motor.dae"/>
+		   </geometry>
+		   </xacro:if>
+		   <xacro:unless value="${hq}">
+		   <geometry>
+		   <mesh filename="package://rb1_arm_description/meshes/arms/armRB1_1_motor.stl"/>
+		   </geometry>
+		   </xacro:unless>
+		   <material name="darkgrey">
+			 <color rgba="0.1 0.1 0.1 1"/>
+		   </material>
+		</visual>
+		<collision>
+		   <origin xyz="0 0 0" rpy="0 0 0 " />
+		   <geometry>
+			 <mesh filename="package://rb1_arm_description/meshes/arms/armRB1_1_motor.dae"/>
+		   </geometry>
+		</collision>
+	</link>
+	<joint
+		name="j01m_rb1_arm"
+		type="fixed">
+		<origin
+		  xyz="0.0 0.0 0.0"
+		  rpy="0.0 0.0 0.0" />
+		<parent
+		  link="link01_rb1_arm" />
+		<child
+		  link="motor01_rb1_arm" />
+		<axis
+		  xyz="0 0 0" />
+	</joint>
+    <!-- JOINT 1 -->
+    <link name="link12_rb1_arm">
+		<inertial>
+		  <mass value="0.7" />
+		  <origin xyz="0.07155 0.00229 -0.00028" />
+		  <inertia  ixx="0.0018430902" ixy="0.0001075379"  ixz="2.683183e-005"  iyy="0.0023530852"  iyz="4.5192e-007"  izz="0.0016327528" />
+		</inertial>
+		<visual>
+		   <origin xyz="0 0 0" rpy="0 0 0" />
+		   <xacro:if value="${hq}">
+		   <geometry>
+			 <mesh filename="package://rb1_arm_description/meshes/arms/armRB1_12_link.dae"/>
+		   </geometry>
+		   </xacro:if>
+		   <xacro:unless value="${hq}">
+		   <geometry>
+		   <mesh filename="package://rb1_arm_description/meshes/arms/armRB1_12_link.stl"/>
+		   </geometry>
+		   </xacro:unless>
+		   <material name="darkgrey">
+			 <color rgba="0.1 0.1 0.1 1"/>
+		   </material>
+		</visual>
+		<collision>
+		   <origin xyz="0 0 0" rpy="0 0 0 " />
+		   <geometry>
+			 <mesh filename="package://rb1_arm_description/meshes/arms/armRB1_12_link.dae"/>
+		   </geometry>
+		</collision>
+	</link>
+	<link name="motor12_rb1_arm">
+		<inertial>
+		  <mass value="0.855" />
+		  <origin xyz="0.13488 -0.00693 0" />
+		  <inertia ixx="0.001211476" ixy="-6.05332e-006" ixz="0.0" iyy="0.0003787678" iyz="0.0" izz="0.001211334"/>
+		</inertial>
+		<visual>
+		   <origin xyz="0 0 0" rpy="0 0 0" />
+		   <xacro:if value="${hq}">
+		   <geometry>
+			 <mesh filename="package://rb1_arm_description/meshes/arms/armRB1_12_motor.dae"/>
+		   </geometry>
+		   </xacro:if>
+		   <xacro:unless value="${hq}">
+		   <geometry>
+		   <mesh filename="package://rb1_arm_description/meshes/arms/armRB1_12_motor.stl"/>
+		   </geometry>
+		   </xacro:unless>
+		   <material name="darkgrey">
+			 <color rgba="0.1 0.1 0.1 1"/>
+		   </material>
+		</visual>
+		<collision>
+		   <origin xyz="0 0 0" rpy="0 0 0 " />
+		   <geometry>
+			 <mesh filename="package://rb1_arm_description/meshes/arms/armRB1_12_motor.dae"/>
+		   </geometry>
+		</collision>
+	</link>
+	<joint
+		name="j12m_rb1_arm"
+		type="fixed">
+		<origin
+		  xyz="0.0 0.0 0.0"
+		  rpy="0.0 0.0 0.0" />
+		<parent
+		  link="link12_rb1_arm" />
+		<child
+		  link="motor12_rb1_arm" />
+		<axis
+		  xyz="0 0 0" />
 	</joint>
 	<joint
 		name="j1"
 		type="revolute">
-	  <origin
-        xyz="0 0 0"
-        rpy="0.0 0.0 0.0" />
-	  <parent link="link1_rb1_arm" />
-      <child link="link12_rb1_arm" />
-      <axis xyz="0 0 -1" />
-      <limit effort="${joint_effort_limit}" velocity="${joint_velocity_limit}" upper="${PI/2}" lower="${-PI/2}"/>
-      <dynamics damping="${joint_damping}" friction="${joint_friction}"/>
-    </joint>
+		<origin
+			xyz="0 0 0"
+			rpy="0.0 0.0 0.0" />
+		<parent link="link01_rb1_arm" />
+		<child link="link12_rb1_arm" />
+		<axis xyz="0 0 -1" />
+		<limit effort="${joint_effort_limit_H54_200}" velocity="${joint_velocity_limit_H54_200}" upper="${j1_upper_limit}" lower="${j1_lower_limit}"/>
+		<dynamics damping="${joint_damping}" friction="${joint_friction}"/>
+	</joint>
     <transmission name="j1_trans">
 	 <type>transmission_interface/SimpleTransmission</type>
@@ -69,4 +224,77 @@
 	 </actuator>
     </transmission>
+    <!-- JOINT 2 -->
+	<link name="link23_rb1_arm">
+		<inertial>
+		  <mass value="0.429" />
+		  <origin xyz="0.06076 0 -0.00014" />
+		  <inertia  ixx="0.0011551458" ixy="-6.3e-010"  ixz="2.519546e-005"  iyy="0.0015754353"  iyz="-7.6e-010"  izz="0.0007798411" />
+		</inertial>
+		<visual>
+		   <origin xyz="0 0 0" rpy="0 0 0" />
+		   <xacro:if value="${hq}">
+		   <geometry>
+			 <mesh filename="package://rb1_arm_description/meshes/arms/armRB1_23_link.dae"/>
+		   </geometry>
+		   </xacro:if>
+		   <xacro:unless value="${hq}">
+		   <geometry>
+		   <mesh filename="package://rb1_arm_description/meshes/arms/armRB1_23_link.stl"/>
+		   </geometry>
+		   </xacro:unless>
+		   <material name="darkgrey">
+			 <color rgba="0.1 0.1 0.1 1"/>
+		   </material>
+		</visual>
+		<collision>
+		   <origin xyz="0 0 0" rpy="0 0 0 " />
+		   <geometry>
+			 <mesh filename="package://rb1_arm_description/meshes/arms/armRB1_23_link.dae"/>
+		   </geometry>
+		</collision>
+	</link>
+	<link name="motor23_rb1_arm">
+		<inertial>
+		  <mass value="0.732" />
+		  <origin xyz="0.11598 0 0.00014" />
+		  <!--inertia  ixx="0.01" ixy="0.0"  ixz="0.0"  iyy="0.01"  iyz="0.0"  izz="0.01" /-->
+		  <inertia ixx="0.02661733557" ixy="0.00029270634" ixz="0.00392189887" iyy="0.02844355207" iyz="0.0010838933" izz="0.01248008322"/>
+		</inertial>
+		<visual>
+		   <origin xyz="0 0 0" rpy="0 0 0" />
+		   <xacro:if value="${hq}">
+		   <geometry>
+			 <mesh filename="package://rb1_arm_description/meshes/arms/armRB1_23_motor.dae"/>
+		   </geometry>
+		   </xacro:if>
+		   <xacro:unless value="${hq}">
+		   <geometry>
+		   <mesh filename="package://rb1_arm_description/meshes/arms/armRB1_23_motor.stl"/>
+		   </geometry>
+		   </xacro:unless>
+		   <material name="darkgrey">
+			 <color rgba="0.1 0.1 0.1 1"/>
+		   </material>
+		</visual>
+		<collision>
+		   <origin xyz="0 0 0" rpy="0 0 0 " />
+		   <geometry>
+			 <mesh filename="package://rb1_arm_description/meshes/arms/armRB1_23_motor.dae"/>
+		   </geometry>
+		</collision>
+	</link>
+	<joint
+		name="j23m_rb1_arm"
+		type="fixed">
+		<origin
+		  xyz="0.0 0.0 0.0"
+		  rpy="0.0 0.0 0.0" />
+		<parent
+		  link="link23_rb1_arm" />
+		<child
+		  link="motor23_rb1_arm" />
+		<axis
+		  xyz="0 0 0" />
+	</joint>
 	<joint
 		name="j2"
@@ -78,5 +306,5 @@
       <child link="link23_rb1_arm" />
       <axis xyz="0 0 -1" />
-      <limit effort="${joint_effort_limit}" velocity="${joint_velocity_limit}" upper="${PI/2}" lower="${-PI/2}"/>
+      <limit effort="${joint_effort_limit_H54_200}" velocity="${joint_velocity_limit_H54_200}" upper="${j2_upper_limit}" lower="${j2_lower_limit}"/>
       <dynamics damping="${joint_damping}" friction="${joint_friction}"/>
     </joint>
@@ -90,4 +318,76 @@
 	 </actuator>
     </transmission>
+    <!-- JOINT 3 -->
+   <link name="link34_rb1_arm">
+		<inertial>
+		  <mass value="0.351" />
+		  <origin xyz="-0.07306 0 -0.00466" />
+		  <inertia  ixx="0.0003749308" ixy="0.0"  ixz="-0.0001258961"  iyy="0.0010047174"  iyz="0.0"  izz="0.0009318091" />
+		</inertial>
+		<visual>
+		   <origin xyz="0 0 0" rpy="0 0 0" />
+		   <xacro:if value="${hq}">
+		   <geometry>
+			 <mesh filename="package://rb1_arm_description/meshes/arms/armRB1_34_link.dae"/>
+		   </geometry>
+		   </xacro:if>
+		   <xacro:unless value="${hq}">
+		   <geometry>
+		   <mesh filename="package://rb1_arm_description/meshes/arms/armRB1_34_link.stl"/>
+		   </geometry>
+		   </xacro:unless>
+		   <material name="darkgrey">
+			 <color rgba="0.1 0.1 0.1 1"/>
+		   </material>
+		</visual>
+		<collision>
+		   <origin xyz="0 0 0" rpy="0 0 0 " />
+		   <geometry>
+			 <mesh filename="package://rb1_arm_description/meshes/arms/armRB1_34_link.dae"/>
+		   </geometry>
+		</collision>
+	</link>
+	<link name="motor34_rb1_arm">
+		<inertial>
+		  <mass value="0.732" />
+		  <origin xyz="0.00014 0 0.00698" />
+		  <inertia ixx="0.0007977173" ixy="0.0" ixz="-5.17658e-006" iyy="0.000797409" iyz="0.0" izz="0.0003233065"/>
+		</inertial>
+		<visual>
+		   <origin xyz="0 0 0" rpy="0 0 0" />
+		   <xacro:if value="${hq}">
+		   <geometry>
+			 <mesh filename="package://rb1_arm_description/meshes/arms/armRB1_34_motor.dae"/>
+		   </geometry>
+		   </xacro:if>
+		   <xacro:unless value="${hq}">
+		   <geometry>
+		   <mesh filename="package://rb1_arm_description/meshes/arms/armRB1_34_motor.stl"/>
+		   </geometry>
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
File: rb1_arm_description/urdf/grippers/two_finger_gripper.urdf.xacro (robot description, xacro)
@@ -3,4 +3,8 @@
   <xacro:property name="finger_mechanical_reduction" value="304.0"/>
   <xacro:property name="finger_motor_torque_constant" value="3.0"/>
+  <xacro:property name="joint_effort_limit" value="3.0"/>
+  <xacro:property name="joint_velocity_limit" value="2.98452"/>
+	<xacro:property name="finger_lower_limit" value="-0.5"/>
+	<xacro:property name="finger_upper_limit" value="0.5"/>
   <xacro:include filename="$(find rb1_arm_description)/urdf/grippers/two_finger_gripper.gazebo.xacro" />
   <link
@@ -97,5 +101,5 @@
     <axis
       xyz="0 0 -1" />
-    <limit effort="${joint_effort_limit}" velocity="${joint_velocity_limit}" upper="1.0" lower="-1.0"/>
+    <limit effort="${joint_effort_limit}" velocity="${joint_velocity_limit}" upper="${finger_upper_limit}" lower="${finger_lower_limit}"/>
     <dynamics damping="${joint_damping}" friction="${joint_friction}"/>
   </joint>
@@ -160,6 +164,6 @@
       link="link_finger2" />
     <axis
-      xyz="0 0 -1" />
-    <limit effort="${joint_effort_limit}" velocity="${joint_velocity_limit}" upper="1.0" lower="-1.0"/>
+      xyz="0 0 1" />
+    <limit effort="${joint_effort_limit}" velocity="${joint_velocity_limit}" upper="${finger_upper_limit}" lower="${finger_lower_limit}"/>
     <dynamics damping="${joint_damping}" friction="${joint_friction}"/>
   </joint>

File: rb1_arm_description/urdf/links/rb1_arm_link.urdf.xacro (robot description, xacro)
@@ -35,5 +35,6 @@
       <mass value="0.5" />
       <origin xyz="0 0 0" />
-      <inertia  ixx="0.01" ixy="0.0"  ixz="0.0"  iyy="0.01"  iyz="0.0"  izz="0.01" />
+      <!--inertia  ixx="0.01" ixy="0.0"  ixz="0.0"  iyy="0.01"  iyz="0.0"  izz="0.01" /-->
+      <inertia ixx="0.02661733557" ixy="0.00029270634" ixz="0.00392189887" iyy="0.02844355207" iyz="0.0010838933" izz="0.01248008322"/>
     </inertial>
     <visual>

File: rb1_torso_description/urdf/rb1_torso_3dof.urdf.xacro (robot description, xacro)
@@ -4,4 +4,6 @@
   <xacro:property name="joint_effort_limit" value="100.0"/>
   <xacro:property name="joint_velocity_limit" value="3.0"/>
+  <xacro:property name="joint_effort_limit_torso" value="5000.0"/>
+  <xacro:property name="joint_velocity_limit_torso" value="1.0"/>
   <xacro:property name="joint_damping" value="0.5"/>
   <xacro:property name="joint_friction" value="0.5"/>
@@ -99,5 +101,5 @@
     <child link="link2_torso" />
     <axis xyz="0 0 1" />
-    <limit effort="${joint_effort_limit}" velocity="${joint_velocity_limit}" upper="${0.360}" lower="${0}"/>
+    <limit effort="${joint_effort_limit_torso}" velocity="${joint_velocity_limit_torso}" upper="${0.360}" lower="${0}"/>
     <dynamics damping="${joint_damping}" friction="${joint_friction}"/>
   </joint>
