Commit message: updated arm urdfs

File: rb1_arm_description/urdf/arms/rb1_arm_7dof.urdf.xacro (robot description, xacro)
@@ -4,7 +4,7 @@
   <xacro:include filename="$(find rb1_arm_description)/urdf/links/rb1_arm_link.urdf.xacro" />
   <xacro:property name="j1_mechanical_reduction" value="502.0"/>
-  <xacro:property name="j1_motor_torque_constant" value="5.0"/>
+  <xacro:property name="j1_motor_torque_constant" value="50.0"/>
   <xacro:property name="j2_mechanical_reduction" value="502.0"/>
-  <xacro:property name="j2_motor_torque_constant" value="5.0"/>
+  <xacro:property name="j2_motor_torque_constant" value="50.0"/>
   <xacro:property name="j3_mechanical_reduction" value="502.0"/>
   <xacro:property name="j3_motor_torque_constant" value="5.0"/>
@@ -17,12 +17,11 @@
   <xacro:property name="j7_mechanical_reduction" value="304.0"/>
   <xacro:property name="j7_motor_torque_constant" value="3.0"/>
-  <xacro:property name="joint_effort_limit" value="100.0"/>
+  <xacro:property name="joint_effort_limit" value="2500.0"/>
   <xacro:property name="joint_velocity_limit" value="3.0"/>
-  <xacro:property name="joint_damping" value="0.5"/>
-  <xacro:property name="joint_friction" value="0.5"/>
+  <xacro:property name="joint_damping" value="0.1"/>
+  <xacro:property name="joint_friction" value="0.1"/>
   <xacro:macro name="rb1_arm_7dof" params="name hq">
     <!-- Robot mechanical and motor parameters -->
     <xacro:property name="PI" value="3.1415926535897931"/>
-    <xacro:property name="gearbox" value="500.0" />
     <!-- BASE_LINK -->
     <link
@@ -175,6 +174,25 @@
 	 </actuator>
     </transmission>
-    <link
-      name="end_effector_rb1_arm">
+    <link name="end_effector_rb1_arm">
+	    <visual>
+		  <origin xyz="0 0 0" rpy="0 0 0" />
+		  <geometry>
+			<cylinder length="0.010" radius="0.025"/>
+		  </geometry>
+		</visual>
+		<collision>
+		  <origin xyz="0 0 0" rpy="0 0 0" />
+		  <geometry>
+			<cylinder length="0.010" radius="0.025"/>
+		  </geometry>
+		</collision>
+		<inertial>
+		  <origin xyz="0 0 0" rpy="0 0 0" />
+		  <mass value="0.1" />
+			<inertia
+			  ixx="0.01" ixy="0.0" ixz="0.0"
+			  iyy="0.01" iyz="0.0"
+			  izz="0.01" />
+		</inertial>
     </link>
 	<joint
@@ -183,5 +201,5 @@
 	  <origin
         xyz="0 0 0"
-        rpy="0.0 0.0 0.0" />
+        rpy="0.0 ${PI/2} 0.0" />
 	  <parent link="link67_rb1_arm" />
       <child link="end_effector_rb1_arm" />

File: rb1_arm_description/urdf/links/rb1_arm_link.urdf.xacro (robot description, xacro)
@@ -4,7 +4,7 @@
   <link name="link${num}_rb1_arm">
     <inertial>
-      <mass value="1.0" />
+      <mass value="0.5" />
       <origin xyz="0 0 0" />
-      <inertia  ixx="1.0" ixy="0.0"  ixz="0.0"  iyy="1.0"  iyz="0.0"  izz="1.0" />
+      <inertia  ixx="0.01" ixy="0.0"  ixz="0.0"  iyy="0.01"  iyz="0.0"  izz="0.01" />
     </inertial>
     <visual>
@@ -33,7 +33,7 @@
   <link name="motor${num}_rb1_arm">
     <inertial>
-      <mass value="1.0" />
+      <mass value="0.5" />
       <origin xyz="0 0 0" />
-      <inertia  ixx="1.0" ixy="0.0"  ixz="0.0"  iyy="1.0"  iyz="0.0"  izz="1.0" />
+      <inertia  ixx="0.01" ixy="0.0"  ixz="0.0"  iyy="0.01"  iyz="0.0"  izz="0.01" />
     </inertial>
     <visual>

Commit message: updated arm urdf

File: rb1_arm_description/urdf/arms/rb1_arm_7dof.urdf.xacro (robot description, xacro)
@@ -99,5 +99,5 @@
       <child link="link34_rb1_arm" />
       <axis xyz="1 0 0" />
-      <limit effort="${joint_effort_limit}" velocity="${joint_velocity_limit}" upper="${PI/2}" lower="${-PI/2}"/>
+      <limit effort="${joint_effort_limit}" velocity="${joint_velocity_limit}" upper="${PI}" lower="${-PI}"/>
       <dynamics damping="${joint_damping}" friction="${joint_friction}"/>
     </joint>
@@ -120,5 +120,5 @@
       <child link="link45_rb1_arm" />
       <axis xyz="0 0 -1" />
-      <limit effort="${joint_effort_limit}" velocity="${joint_velocity_limit}" upper="${PI/2}" lower="${-PI/2}"/>
+      <limit effort="${joint_effort_limit}" velocity="${joint_velocity_limit}" upper="${2.0}" lower="${-2.0}"/>
       <dynamics damping="${joint_damping}" friction="${joint_friction}"/>
     </joint>
@@ -141,5 +141,5 @@
       <child link="link56_rb1_arm" />
       <axis xyz="1 0 0" />
-      <limit effort="${joint_effort_limit}" velocity="${joint_velocity_limit}" upper="${PI/2}" lower="${-PI/2}"/>
+      <limit effort="${joint_effort_limit}" velocity="${joint_velocity_limit}" upper="${PI}" lower="${-PI}"/>
       <dynamics damping="${joint_damping}" friction="${joint_friction}"/>
     </joint>
@@ -162,5 +162,5 @@
       <child link="link67_rb1_arm" />
       <axis xyz="0 0 -1" />
-      <limit effort="${joint_effort_limit}" velocity="${joint_velocity_limit}" upper="${PI/2}" lower="${-PI/2}"/>
+      <limit effort="${joint_effort_limit}" velocity="${joint_velocity_limit}" upper="${2.0}" lower="${-2.0}"/>
       <dynamics damping="${joint_damping}" friction="${joint_friction}"/>
     </joint>
@@ -176,7 +176,7 @@
     <link name="end_effector_rb1_arm">
 	    <visual>
-		  <origin xyz="0 0 0" rpy="0 0 0" />
+		  <origin xyz="0 0 0.030" rpy="0 0 0" />
 		  <geometry>
-			<cylinder length="0.010" radius="0.025"/>
+			<cylinder length="0.010" radius="0.015"/>
 		  </geometry>
 		</visual>
@@ -184,5 +184,5 @@
 		  <origin xyz="0 0 0" rpy="0 0 0" />
 		  <geometry>
-			<cylinder length="0.010" radius="0.025"/>
+			<cylinder length="0.005" radius="0.025"/>
 		  </geometry>
 		</collision>
@@ -205,5 +205,5 @@
       <child link="end_effector_rb1_arm" />
       <axis xyz="0 0 -1" />
-      <limit effort="${joint_effort_limit}" velocity="${joint_velocity_limit}" upper="${PI/2}" lower="${-PI/2}"/>
+      <limit effort="${joint_effort_limit}" velocity="${joint_velocity_limit}" upper="${PI}" lower="${-PI}"/>
       <dynamics damping="${joint_damping}" friction="${joint_friction}"/>
     </joint>

Commit message: state robot launch added, and updated rotation signs

File: rb1_arm_description/urdf/arms/rb1_arm_7dof.urdf.xacro (robot description, xacro)
@@ -211,5 +211,5 @@
 		<parent link="link01_rb1_arm" />
 		<child link="link12_rb1_arm" />
-		<axis xyz="0 0 -1" />
+		<axis xyz="0 0 1" />
 		<limit effort="${joint_effort_limit_H54_200}" velocity="${joint_velocity_limit_H54_200}" upper="${j1_upper_limit}" lower="${j1_lower_limit}"/>
 		<dynamics damping="${joint_damping}" friction="${joint_friction}"/>
@@ -305,5 +305,7 @@
 	  <parent link="link12_rb1_arm" />
       <child link="link23_rb1_arm" />
-      <axis xyz="0 0 -1" />
+      <!-- check -->
+      <!-- axis xyz="0 0 -1" / -->
+      <axis xyz="0 0 1"/>
       <limit effort="${joint_effort_limit_H54_200}" velocity="${joint_velocity_limit_H54_200}" upper="${j2_upper_limit}" lower="${j2_lower_limit}"/>
       <dynamics damping="${joint_damping}" friction="${joint_friction}"/>
@@ -491,5 +493,7 @@
 	  <parent link="link34_rb1_arm" />
       <child link="link45_rb1_arm" />
-      <axis xyz="0 0 -1" />
+      <!-- check -->
+      <!-- xis xyz="0 0 -1" / -->
+      <axis xyz="0 0 1"/>
       <limit effort="${joint_effort_limit_H54_100}" velocity="${joint_velocity_limit_H54_100}" upper="${j4_upper_limit}" lower="${j4_lower_limit}"/>
       <dynamics damping="${joint_damping}" friction="${joint_friction}"/>
@@ -677,5 +681,7 @@
 	  <parent link="link56_rb1_arm" />
       <child link="link67_rb1_arm" />
-      <axis xyz="0 0 -1" />
+      <!-- check -->
+      <!-- axis xyz="0 0 -1" / -->
+      <axis xyz="0 0 1"/>
       <limit effort="${joint_effort_limit_L42}" velocity="${joint_velocity_limit_L42}" upper="${j6_upper_limit}" lower="${j6_lower_limit}"/>
       <dynamics damping="${joint_damping}" friction="${joint_friction}"/>
@@ -694,5 +700,5 @@
 	  <origin
         xyz="0 0 0"
-        rpy="0.0 0.0 0.0" />
+        rpy="1.5708 0.0 0.0" />
 	  <parent link="link67_rb1_arm" />
       <child link="end_effector_rb1_arm" />

File: rb1_torso_description/urdf/rb1_torso_3dof.urdf.xacro (robot description, xacro)
@@ -200,5 +200,7 @@
 	<parent link="link1_head" />
     <child link="link2_head" />
-    <axis xyz="0 1 0" />
+    <!-- check -->
+    <!-- axis xyz="0 1 0" / -->
+    <axis xyz="0 -1 0"/>
     <limit effort="${joint_effort_limit}" velocity="${joint_velocity_limit}" upper="${PI/4}" lower="${-PI/4}"/>
     <dynamics damping="${joint_damping}" friction="${joint_friction}"/>

Commit message: updated urdf ranges to real limits

File: rb1_arm_description/urdf/arms/rb1_arm_7dof.urdf.xacro (robot description, xacro)
@@ -16,16 +16,16 @@
 	<xacro:property name="j7_mechanical_reduction" value="304.0"/>
 	<xacro:property name="j7_motor_torque_constant" value="3.0"/>
-	<xacro:property name="j1_lower_limit" value="-1.570796327"/>
-	<xacro:property name="j1_upper_limit" value="1.570796327"/>
-	<xacro:property name="j2_lower_limit" value="-1.570796327"/>
-	<xacro:property name="j2_upper_limit" value="1.570796327"/>
+	<xacro:property name="j1_lower_limit" value="-1.55"/>
+	<xacro:property name="j1_upper_limit" value="1.55"/>
+	<xacro:property name="j2_lower_limit" value="-1.95"/>
+	<xacro:property name="j2_upper_limit" value="1.55"/>
 	<xacro:property name="j3_lower_limit" value="-3.13"/>
 	<xacro:property name="j3_upper_limit" value="3.13"/>
-	<xacro:property name="j4_lower_limit" value="-1.570796327"/>
-	<xacro:property name="j4_upper_limit" value="1.570796327"/>
+	<xacro:property name="j4_lower_limit" value="-1.95"/>
+	<xacro:property name="j4_upper_limit" value="1.95"/>
 	<xacro:property name="j5_lower_limit" value="-3.13"/>
 	<xacro:property name="j5_upper_limit" value="3.13"/>
-	<xacro:property name="j6_lower_limit" value="-1.570796327"/>
-	<xacro:property name="j6_upper_limit" value="1.570796327"/>
+	<xacro:property name="j6_lower_limit" value="-1.57"/>
+	<xacro:property name="j6_upper_limit" value="1.57"/>
 	<xacro:property name="j7_lower_limit" value="-3.13"/>
 	<xacro:property name="j7_upper_limit" value="3.13"/>
