Commit message: description changes for standalone / rb1 sim

File: rb1_description/robots/rb1_robot.urdf (robot description, URDF)
Before this commit: robot rb1, 31 links, 28 joints
Links:
- removed link base_footprint
- removed link base_link
- removed link link1_head_rb1_torso
- removed link link1_rb1_torso
- removed link link2_head_rb1_torso
- removed link link2_rb1_torso
- added link base_link_gripper, mass 0.2735; collision mesh filename=package://rb1_arm_description/meshes/grippers/base_gripper.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; visual mesh filename=package://rb1_arm_description/meshes/grippers/base_gripper.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
- added link link1_head, mass 1.0; collision mesh filename=package://rb1_torso_description/meshes/heads/head1.dae; visual mesh filename=package://rb1_torso_description/meshes/heads/head1.dae
- added link link1_torso, mass 3.0; collision mesh filename=package://rb1_torso_description/meshes/torsos/rb1_lower.dae; visual mesh filename=package://rb1_torso_description/meshes/torsos/rb1_lower.dae
- added link link2_head, mass 1.0; collision mesh filename=package://rb1_torso_description/meshes/heads/head2.dae; visual mesh filename=package://rb1_torso_description/meshes/heads/head2.dae
- added link link2_torso, mass 2.0; collision mesh filename=package://rb1_torso_description/meshes/torsos/rb1_upper.dae; visual mesh filename=package://rb1_torso_description/meshes/torsos/rb1_upper.dae
- added link link_finger1, mass 0.03; collision mesh filename=package://rb1_arm_description/meshes/grippers/finger1.dae; visual mesh filename=package://rb1_arm_description/meshes/grippers/finger1.dae
- added link link_finger2, mass 0.03; collision mesh filename=package://rb1_arm_description/meshes/grippers/finger2.dae; visual mesh filename=package://rb1_arm_description/meshes/grippers/finger2.dae
- added link xtion_head_cam_depth_frame, mass 0.01
- added link xtion_head_cam_depth_optical_frame, mass 0.001
- added link xtion_head_cam_link, mass 0.01; collision box size=0.0730 .2760 0.0720; visual mesh filename=package://rb1_base_description/meshes/sensors/asus_xtion_pr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 scale=0.001 0.001 0.001
- added link xtion_head_cam_rgb_frame, mass 0.001
- added link xtion_head_cam_rgb_optical_frame, mass 0.001
- link end_effector_rb1_arm: mass None -> 0.1; geometry collision cylinder length=0.005 radius=0.025; visual cylinder length=0.010 radius=0.015
- link link12_rb1_arm: mass 1.0 -> 0.5
- link link1_rb1_arm: mass 1.0 -> 0.5
- link link23_rb1_arm: mass 1.0 -> 0.5
- link link34_rb1_arm: mass 1.0 -> 0.5
- link link45_rb1_arm: mass 1.0 -> 0.5
- link link56_rb1_arm: mass 1.0 -> 0.5
- link link67_rb1_arm: mass 1.0 -> 0.5
- link motor12_rb1_arm: mass 1.0 -> 0.5
- link motor1_rb1_arm: mass 1.0 -> 0.5
- link motor23_rb1_arm: mass 1.0 -> 0.5
- link motor34_rb1_arm: mass 1.0 -> 0.5
- link motor45_rb1_arm: mass 1.0 -> 0.5
- link motor56_rb1_arm: mass 1.0 -> 0.5
- link motor67_rb1_arm: mass 1.0 -> 0.5
Joints:
- removed joint base_footprint_joint
- removed joint j1_head_rb1_torso
- removed joint j1_rb1_torso
- removed joint j2_head_rb1_torso
- added joint gripper_joint: type fixed, parent end_effector_rb1_arm, child base_link_gripper, origin xyz=0.0 0.0 0.0 rpy=0.0 -1.57079632679 0.0, axis 0 0 1
- added joint j1_head: type revolute, parent link2_torso, child link1_head, origin xyz=0.010 0.0 0.940 rpy=0.0 0.0 0.0, axis 0 0 1, limit lower=-1.57079632679 upper=1.57079632679 effort=2500.0 velocity=3.0
- added joint j1_torso: type prismatic, parent link1_torso, child link2_torso, origin xyz=0 0 0 rpy=0.0 0.0 0.0, axis 0 0 1, limit lower=0.0 upper=0.36 effort=2500.0 velocity=3.0
- added joint j2_head: type revolute, parent link1_head, child link2_head, origin xyz=0.105 0.0 0.0 rpy=0.0 0.0 0.0, axis 0 1 0, limit lower=-0.785398163397 upper=0.785398163397 effort=2500.0 velocity=3.0
- added joint j_base_torso: type fixed, parent base_link, child base_link_rb1_torso, origin xyz=0.0 0.0 0.0 rpy=0.0 0.0 0.0, axis 0 0 0
- added joint j_torso_arm: type fixed, parent link2_torso, child base_link_rb1_arm, origin xyz=0.074 0.0 0.668 rpy=0.0 0.0 0.0, axis 0 0 0
- added joint jg1: type revolute, parent base_link_gripper, child link_finger1, origin xyz=0.097993 0.028575 0 rpy=3.0028E-16 5.9154E-22 2.2204E-16, axis 0 0 -1, limit lower=-1.0 upper=1.0 effort=2500.0 velocity=3.0
- added joint jg2: type revolute, parent base_link_gripper, child link_finger2, origin xyz=0.097993 -0.028575 0 rpy=3.0028E-16 7.477E-22 -5.1764E-15, axis 0 0 -1, limit lower=-1.0 upper=1.0 effort=2500.0 velocity=3.0
- added joint xtion_head_cam_depth_joint: type fixed, parent xtion_head_cam_rgb_frame, child xtion_head_cam_depth_frame, origin xyz=0 0.027 0 rpy=0 0 0
- added joint xtion_head_cam_depth_optical_joint: type fixed, parent xtion_head_cam_depth_frame, child xtion_head_cam_depth_optical_frame, origin xyz=0 0 0 rpy=-1.57079632679 0 -1.57079632679
- added joint xtion_head_cam_joint: type fixed, parent xtion_head_cam_rgb_frame, child xtion_head_cam_link, origin xyz=0 -0.022 0 rpy=0 0 0
- added joint xtion_head_cam_rgb_joint: type fixed, parent link2_head, child xtion_head_cam_rgb_frame, origin xyz=0.055 0.000 0.028 rpy=0 0 0
- added joint xtion_head_cam_rgb_optical_joint: type fixed, parent xtion_head_cam_rgb_frame, child xtion_head_cam_rgb_optical_frame, origin xyz=0 0 0 rpy=-1.57079632679 0 -1.57079632679
- joint j0_rb1_torso: child link1_rb1_torso -> link1_torso
- joint j1: limit lower=-1.57079632679 upper=1.57079632679 effort=100.0 velocity=3.0 -> lower=-1.57079632679 upper=1.57079632679 effort=2500.0 velocity=3.0
- joint j2: limit lower=-1.57079632679 upper=1.57079632679 effort=100.0 velocity=3.0 -> lower=-1.57079632679 upper=1.57079632679 effort=2500.0 velocity=3.0
- joint j3: limit lower=-1.57079632679 upper=1.57079632679 effort=100.0 velocity=3.0 -> lower=-3.14159265359 upper=3.14159265359 effort=2500.0 velocity=3.0
- joint j4: limit lower=-1.57079632679 upper=1.57079632679 effort=100.0 velocity=3.0 -> lower=-2.0 upper=2.0 effort=2500.0 velocity=3.0
- joint j5: limit lower=-1.57079632679 upper=1.57079632679 effort=100.0 velocity=3.0 -> lower=-3.14159265359 upper=3.14159265359 effort=2500.0 velocity=3.0
- joint j6: limit lower=-1.57079632679 upper=1.57079632679 effort=100.0 velocity=3.0 -> lower=-2.0 upper=2.0 effort=2500.0 velocity=3.0
- joint j7: limit lower=-1.57079632679 upper=1.57079632679 effort=100.0 velocity=3.0 -> lower=-3.14159265359 upper=3.14159265359 effort=2500.0 velocity=3.0; origin xyz=0 0 0 rpy=0.0 0.0 0.0 -> xyz=0 0 0 rpy=0.0 1.57079632679 0.0

File: rb1_description/robots/rb1_robot.urdf.xacro (robot description, xacro)
@@ -12,5 +12,5 @@
 	<xacro:include filename="$(find rb1_arm_description)/robots/rb1_arm.urdf.xacro" />
 	<!-- Gazebo ros control plugins -->
-	<xacro:ros_control/>
+	<!-- xacro:ros_control/ -->
 	<!-- Fix torso to base -->
 	<joint

Commit message: updated urdf

File: rb1_description/robots/rb1_robot.urdf (robot description, URDF)
Before this commit: robot rb1, 37 links, 37 joints
Links:
- added link base_footprint; visual box size=0.001 0.001 0.001
- added link base_link, mass 25.0; collision mesh filename=package://rb1_base_description/meshes/bases/rb1_base.dae; visual mesh filename=package://rb1_base_description/meshes/bases/rb1_base.dae
Joints:
- added joint base_footprint_joint: type fixed, parent base_footprint, child base_link, origin xyz=0 0 0.025 rpy=0 0 0

Commit message: updated rb1_robot.urdf

File: rb1_description/robots/rb1_robot.urdf (robot description, URDF)
Before this commit: robot rb1, 39 links, 38 joints
Links:
- removed link hokuyo1_laser_link
- removed link link1_rb1_arm
- removed link motor1_rb1_arm
- added link link01_rb1_arm, mass 0.506; collision mesh filename=package://rb1_arm_description/meshes/arms/armRB1_1_link.dae; visual mesh filename=package://rb1_arm_description/meshes/arms/armRB1_1_link.dae
- added link motor01_rb1_arm, mass 0.855; collision mesh filename=package://rb1_arm_description/meshes/arms/armRB1_1_motor.dae; visual mesh filename=package://rb1_arm_description/meshes/arms/armRB1_1_motor.dae
- link base_link_gripper: mass 0.2735 -> 0.257; geometry collision mesh filename=package://rb1_arm_description/meshes/grippers/v1/gripper_mo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; visual mesh filename=package://rb1_arm_description/meshes/grippers/v1/gripper_mo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
- link end_effector_rb1_arm: mass 0.1 -> None; geometry 
- link hokuyo_laser_link: geometry collision box size=0.1 0.1 0.08; visual mesh filename=package://rb1_base_description/meshes/sensors/hokuyo_urg_04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
- link link12_rb1_arm: mass 0.5 -> 0.7
- link link23_rb1_arm: mass 0.5 -> 0.429
- link link34_rb1_arm: mass 0.5 -> 0.351
- link link45_rb1_arm: mass 0.5 -> 0.388
- link link56_rb1_arm: mass 0.5 -> 0.3559
- link link67_rb1_arm: mass 0.5 -> 0.055
- link link_finger1: mass 0.03 -> 0.1264; geometry collision mesh filename=package://rb1_arm_description/meshes/grippers/v1/gripper_li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; visual mesh filename=package://rb1_arm_description/meshes/grippers/v1/gripper_li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
- link link_finger2: mass 0.03 -> 0.0633; geometry collision mesh filename=package://rb1_arm_description/meshes/grippers/v1/gripper_li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; visual mesh filename=package://rb1_arm_description/meshes/grippers/v1/gripper_li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
- link motor12_rb1_arm: mass 0.5 -> 0.855
- link motor23_rb1_arm: mass 0.5 -> 0.732
- link motor34_rb1_arm: mass 0.5 -> 0.732
- link motor45_rb1_arm: mass 0.5 -> 0.732
- link motor56_rb1_arm: mass 0.5 -> 0.34
- link motor67_rb1_arm: mass 0.5 -> 0.34
Joints:
- removed joint hokuyo1_laser_joint
- removed joint j1m_rb1_arm
- added joint j01m_rb1_arm: type fixed, parent link01_rb1_arm, child motor01_rb1_arm, origin xyz=0.0 0.0 0.0 rpy=0.0 0.0 0.0, axis 0 0 0
- joint gripper_joint: axis 0 0 1 -> 1 0 0; origin xyz=0.0 0.0 0.0 rpy=0.0 -1.57079632679 0.0 -> xyz=0.055 0.0 0.0 rpy=0.0 0.0 0.0
- joint hokuyo_laser_joint: origin xyz=0.210 0.0 0.305 rpy=0 0 0 -> xyz=0.220 0.0 0.170 rpy=0 3.1416 3.1416
- joint j1: axis 0 0 -1 -> 0 0 1; limit lower=-1.57079632679 upper=1.57079632679 effort=2500.0 velocity=3.0 -> lower=-1.570796327 upper=1.570796327 effort=60.0 velocity=2.9217; parent link1_rb1_arm -> link01_rb1_arm
- joint j1_head: limit lower=-1.57079632679 upper=1.57079632679 effort=2500.0 velocity=3.0 -> lower=-1.57079632679 upper=1.57079632679 effort=3.0 velocity=2.98452
- joint j1_rb1_arm: child link1_rb1_arm -> link01_rb1_arm
- joint j1_torso: limit lower=0.0 upper=0.36 effort=2500.0 velocity=3.0 -> lower=0.0 upper=0.36 effort=5000.0 velocity=1.0
- joint j2: axis 0 0 -1 -> 0 0 1; limit lower=-1.57079632679 upper=1.57079632679 effort=2500.0 velocity=3.0 -> lower=-1.570796327 upper=1.570796327 effort=60.0 velocity=2.9217
- joint j2_head: axis 0 1 0 -> 0 -1 0; limit lower=-0.785398163397 upper=0.785398163397 effort=2500.0 velocity=3.0 -> lower=-0.785398163397 upper=0.785398163397 effort=3.0 velocity=2.98452
- joint j3: limit lower=-3.14159265359 upper=3.14159265359 effort=2500.0 velocity=3.0 -> lower=-3.13 upper=3.13 effort=35.0 velocity=3.1527
- joint j4: axis 0 0 -1 -> 0 0 1; limit lower=-2.0 upper=2.0 effort=2500.0 velocity=3.0 -> lower=-1.570796327 upper=1.570796327 effort=35.0 velocity=3.1527
- joint j5: limit lower=-3.14159265359 upper=3.14159265359 effort=2500.0 velocity=3.0 -> lower=-3.13 upper=3.13 effort=35.0 velocity=3.1527
- joint j6: axis 0 0 -1 -> 0 0 1; limit lower=-2.0 upper=2.0 effort=2500.0 velocity=3.0 -> lower=-1.570796327 upper=1.570796327 effort=8.0 velocity=2.98452
- joint j7: axis 0 0 -1 -> 1 0 0; limit lower=-3.14159265359 upper=3.14159265359 effort=2500.0 velocity=3.0 -> lower=-3.13 upper=3.13 effort=8.0 velocity=2.98452; origin xyz=0 0 0 rpy=0.0 1.57079632679 0.0 -> xyz=0 0 0 rpy=1.5708 0.0 0.0
- joint jg1: axis 0 0 -1 -> (none); limit lower=-1.0 upper=1.0 effort=2500.0 velocity=3.0 -> (none); origin xyz=0.097993 0.028575 0 rpy=3.0028E-16 5.9154E-22 2.2204E-16 -> xyz=0.0 0.0 0 rpy=0.0 0.0 0.0; type revolute -> fixed
- joint jg2: axis 0 0 -1 -> 0 0 1; limit lower=-1.0 upper=1.0 effort=2500.0 velocity=3.0 -> lower=-0.7 upper=0.0 effort=3.0 velocity=2.98452; origin xyz=0.097993 -0.028575 0 rpy=3.0028E-16 7.477E-22 -5.1764E-15 -> xyz=0.0 0.0 0 rpy=0.0 0.0 0.0
